File: eCAD/humming/humming.sch (EAGLE design)
At the start: 34 parts, among them J1 POWER_JACKPTH_LOCK, U1 LTC6992CS6-1TRMPBF, U2 LM386M-1/NOPB

Commit message: Adding v0.2 pdf
Other:
- note added: "433-1175-ND 433-1171-ND More Expensive: 668-1668-ND 668-1684-ND 668-1691-ND"
- note added: "Some nets are labelled 0 instead of GND. Tie U1 GND to actual GND."
- note removed: "433-1175-ND More Expensive: 668-1668-ND 668-1684-ND 668-1691-ND"
- note removed: "Some nets are labelled 0 instead of GND."
Changed lines of the file:
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@@
 Scale: 0.13</text>
 <text x="256.54" y="68.58" size="1.778" layer="97">433-1175-ND
+433-1171-ND
 More Expensive:
 668-1668-ND
 668-1684-ND
 668-1691-ND</text>
-<text x="48.26" y="152.4" size="1.778" layer="97">Some nets are labelled 0 instead of GND.</text>
+<text x="48.26" y="152.4" size="1.778" layer="97">Some nets are labelled 0 instead of GND.
+Tie U1 GND to actual GND.</text>
 </plain>
 <instances>
@@
 <pinref part="X_1" gate="G$1" pin="0"/>
 <wire x1="38.1" y1="91.44" x2="38.1" y2="88.9" width="0.1524" layer="91"/>
+<label x="40.64" y="88.9" size="1.778" layer="95"/>
 </segment>
 <segment>
@@
 <pinref part="X_3" gate="G$1" pin="0"/>
 <wire x1="99.06" y1="99.06" x2="99.06" y2="96.52" width="0.1524" layer="91"/>
+<label x="101.6" y="96.52" size="1.778" layer="95"/>
 </segment>
 <segment>
@@
 <pinref part="U1" gate="A" pin="GND"/>
 <wire x1="45.72" y1="127" x2="48.26" y2="127" width="0.1524" layer="91"/>
-</segment>
-</net>
+<label x="45.72" y="129.54" size="1.778" layer="95"/>
+</segment>
+</net>
